File: kicad/filament-dryer.kicad_pcb (KiCad board)
At the start: 2 copper layers, 0 parts

Commit message: Component placement done
Parts:
- added BT1: Tactile Button, kicad-ezee-footprints:PushButton-SMD_4P-L5.1-W5.1, F.Cu at (110.5, 57.1)
- added C1: 100n, Capacitor_THT:C_Disc_D4.3mm_W1.9mm_P5.00mm, F.Cu at (91.4, 66.0)
- added C10: 220u, Capacitor_Tantalum_SMD:CP_EIA-6032-28_Kemet-C, F.Cu at (107.4, 40.5)
- added C2: 20p, Capacitor_THT:C_Disc_D4.3mm_W1.9mm_P5.00mm, F.Cu at (84.5, 83.9)
- added C3: 20p, Capacitor_THT:C_Disc_D4.3mm_W1.9mm_P5.00mm, F.Cu at (84.5, 96.5)
- added C4: 15u, Capacitor_Tantalum_SMD:CP_EIA-6032-28_Kemet-C, F.Cu at (90.2, 55.8)
- added C5: 1u, Capacitor_Tantalum_SMD:CP_EIA-6032-20_AVX-F, F.Cu at (88.9, 70.9)
- added C6: 100n, Capacitor_THT:C_Disc_D4.3mm_W1.9mm_P5.00mm, F.Cu at (107.4, 84.9)
- added C7: 100n, Capacitor_THT:C_Disc_D4.3mm_W1.9mm_P5.00mm, F.Cu at (89.8, 80.6)
- added C8: 100n, Capacitor_THT:C_Disc_D4.3mm_W1.9mm_P5.00mm, F.Cu at (107.4, 87.5)
- added C9: 1u, Capacitor_Tantalum_SMD:CP_EIA-6032-20_AVX-F, F.Cu at (110.2, 90.9)
- added CN1: Pololu Mini-LCD, Connector_PinHeader_2.54mm:PinHeader_2x07_P2.54mm_Vertical, F.Cu at (111.7, 78.0)
- added D1: 1N4148, Diode_THT:D_DO-35_SOD27_P7.62mm_Horizontal, F.Cu at (75.6, 74.3)
- added F1: 5A, kicad-ezee-footprints:FuseHolder_20x5mm, F.Cu at (54.0, 87.6)
- added F2: 1A, Fuse:Fuse_1206_3216Metric_Pad1.42x1.75mm_HandSolder, F.Cu at (111.9, 39.3)
- added FID1: 1mm, Fiducial:Fiducial_1mm_Mask2mm, F.Cu at (51.4, 34.9)
- added FID2: 1mm, Fiducial:Fiducial_1mm_Mask2mm, F.Cu at (122.6, 43.8)
- added FID3: 1mm, Fiducial:Fiducial_1mm_Mask2mm, F.Cu at (69.2, 108.6)
- added J1: 24V, kicad-ezee-footprints:TerminalBlock_2_P5.08mm, F.Cu at (55.2, 63.5)
- added J2: AREF_SELECT, Connector_PinHeader_2.54mm:PinHeader_2x02_P2.54mm_Vertical, F.Cu at (109.2, 97.2)
- added J3: Circulation Fan, Connector_PinHeader_2.54mm:PinHeader_1x02_P2.54mm_Vertical, F.Cu at (62.2, 76.8)
- added J4: Fresh Air Fan, Connector_PinHeader_2.54mm:PinHeader_1x02_P2.54mm_Vertical, F.Cu at (74.9, 62.9)
- added J5: AVR-ISP-6, Connector_PinHeader_2.54mm:PinHeader_2x03_P2.54mm_Vertical, F.Cu at (101.6, 104.8)
- added J6: HEATER TEMP, Connector_JST:JST_PH_B2B-PH-K_1x02_P2.00mm_Vertical, F.Cu at (118.0, 72.4)
- added J7: IO, Connector_PinHeader_2.54mm:PinHeader_1x06_P2.54mm_Vertical, F.Cu at (80.6, 64.1)
- added J8: Heater, kicad-ezee-footprints:TerminalBlock_2_P5.08mm, F.Cu at (55.2, 52.7)
- added L1: 68uH, Inductor_SMD:L_12x12mm_H6mm, F.Cu at (97.8, 43.6)
- added MH1: M3, MountingHole:MountingHole_3.2mm_M3_Pad_Via, F.Cu at (44.7, 34.5)
- added MH2: M3, MountingHole:MountingHole_3.2mm_M3_Pad_Via, F.Cu at (44.7, 111.3)
- added MH3: M3, MountingHole:MountingHole_3.2mm_M3_Pad_Via, F.Cu at (128.3, 111.8)
- added MH4: M3, MountingHole:MountingHole_3.2mm_M3_Pad_Via, F.Cu at (128.3, 34.3)
- added Q1: 2N3904, Package_TO_SOT_THT:TO-92_Inline, F.Cu at (70.5, 62.9)
- added Q2: 2N3904, Package_TO_SOT_THT:TO-92_Inline, F.Cu at (75.6, 84.2)
- added Q3: 2N3906, Package_TO_SOT_THT:TO-92_Inline, F.Cu at (75.6, 89.0)
- added Q4: STP75NF75, Package_TO_SOT_THT:TO-220-3_Vertical, F.Cu at (64.1, 101.0)
- added R1: 5.6k, Resistor_THT:R_Axial_DIN0207_L6.3mm_D2.5mm_P10.16mm_Horizontal, F.Cu at (94.0, 59.1)
- added R10: 1.2k, Resistor_THT:R_Axial_DIN0207_L6.3mm_D2.5mm_P10.16mm_Horizontal, F.Cu at (71.8, 88.9)
- added R11: 47k, Resistor_THT:R_Axial_DIN0207_L6.3mm_D2.5mm_P10.16mm_Horizontal, F.Cu at (116.8, 87.0)
- added R12: 4.7k, Resistor_THT:R_Axial_DIN0207_L6.3mm_D2.5mm_P10.16mm_Horizontal, F.Cu at (120.7, 87.0)
- added R13: 100k, Resistor_THT:R_Axial_DIN0207_L6.3mm_D2.5mm_P10.16mm_Horizontal, F.Cu at (71.8, 92.1)
- added R14: 100, Resistor_THT:R_Axial_DIN0207_L6.3mm_D2.5mm_P10.16mm_Horizontal, F.Cu at (61.6, 95.2)
- added R2: 5.6k, Resistor_THT:R_Axial_DIN0207_L6.3mm_D2.5mm_P10.16mm_Horizontal, F.Cu at (116.8, 96.5)
- added R3: 0, Resistor_THT:R_Axial_DIN0207_L6.3mm_D2.5mm_P10.16mm_Horizontal, F.Cu at (120.7, 106.7)
- added R4: 10, Resistor_THT:R_Axial_DIN0207_L6.3mm_D2.5mm_P10.16mm_Horizontal, F.Cu at (94.1, 62.5)
- added R5: 1.2k, Resistor_THT:R_Axial_DIN0207_L6.3mm_D2.5mm_P10.16mm_Horizontal, F.Cu at (69.2, 66.7)
- added R6: 8.2k, Resistor_THT:R_Axial_DIN0207_L6.3mm_D2.5mm_P10.16mm_Horizontal, F.Cu at (72.4, 76.8)
- added R7: 1.2k, Resistor_THT:R_Axial_DIN0207_L6.3mm_D2.5mm_P10.16mm_Horizontal, F.Cu at (80.6, 104.1)
- added R8: 100k, Resistor_THT:R_Axial_DIN0207_L6.3mm_D2.5mm_P10.16mm_Horizontal, F.Cu at (71.8, 82.5)
- added R9: 10k, Resistor_THT:R_Axial_DIN0207_L6.3mm_D2.5mm_P10.16mm_Horizontal, F.Cu at (61.6, 85.7)
- added RV1: 10k, kicad-ezee-footprints:Potentiometer_VANXY_T73YP_Vertical, F.Cu at (118.2, 66.7)
- added TH1: 10k, Resistor_THT:R_Axial_DIN0207_L6.3mm_D2.5mm_P10.16mm_Horizontal, F.Cu at (124.5, 76.8)
- added TJ1: 80 deg, Connector_Wire:SolderWire-0.75sqmm_1x02_P7mm_D1.25mm_OD3.5mm, F.Cu at (57.5, 69.2)
- added U1: ATmega8-16P, Package_DIP:DIP-28_W7.62mm, F.Cu at (95.3, 67.2)
- added U2: MIC4680-5BM, Package_SO:SOIC-8_3.9x4.9mm_P1.27mm, F.Cu at (84.0, 51.5)
- added U3: LM336-2.5, Package_TO_SOT_THT:TO-92L_Inline, F.Cu at (112.3, 105.0)
- added Y1: 16MHz, Crystal:Crystal_HC49-4H_Vertical, F.Cu at (90.2, 92.6)
Other:
- board outline added: 94 x 88.3 mm
- board text removed: "Tips: - Minimum grid : 0.25mm - Theme: Monokai High Contrast"
